File: Daughterboard/Daughterboard_before_nc_smd_pads_removed.kicad_sch (KiCad schematic)
At the start: 153 parts, among them J1 USB-C 5V Sink, J2 Switched power outputs, J30 J3P Hosyond +5V_SW solder pad, J31 J3A Hosyond UART_TX solder pad, J32 J3B Hosyond UART_RX solder pad, J33 J3C Hosyond I2C_SDA solder pad, J34 J3D Hosyond I2C_SCL solder pad, J35 J3E Hosyond GPIO2 solder pad, J36 J3F Hosyond GPIO3 solder pad, J37 J3G Hosyond GPIO14 solder pad, J38 J3H Hosyond GPIO21 solder pad, J39 J3I Hosyond GND solder pad, J4 UART JST-GH 1.25mm, J5 I2C male header 2.54mm, J6 Deep sleep pushbutton header, J7 2S balance input JST-XH, J8 Analog input header, J91 MCP23017 GPA0 solder pad, J910 MCP23017 GPB1 solder pad, J911 MCP23017 GPB2 solder pad, J912 MCP23017 GPB3 solder pad, J913 MCP23017 GPB4 solder pad, J914 MCP23017 GPB5 solder pad, J915 MCP23017 GPB6 solder pad, J916 MCP23017 GPB7 solder pad, J92 MCP23017 GPA1 solder pad, J925 MCP23017 INTA solder pad, J926 MCP23017 INTB solder pad, J927 MCP23017 RESET solder pad, J928 MCP23017 +3V3_SW solder pad, J929 MCP23017 GND solder pad, J93 MCP23017 GPA2 solder pad, J94 MCP23017 GPA3 solder pad, J95 MCP23017 GPA4 solder pad, J96 MCP23017 GPA5 solder pad, J97 MCP23017 GPA6 solder pad, J98 MCP23017 GPA7 solder pad, J99 MCP23017 GPB0 solder pad, Q1 CSD83325L, SW1 Pololu #2808 5V switch, SW2 Pololu #2808 3V3 switch, U1 BQ25887RGE 2S charger, U2 S-8252AAH-M6T1U, U3 AP63200WU 5V Buck, U4 AP63200WU 3V3 Buck, U5 ADS1115IDGS 0x48, U6 ADS1115IDGS 0x49, U7 MCP23017-E/SO

Commit message: a
Parts:
- removed R45: 0R, Resistor_SMD:R_0603_1608Metric, symbol Daughterboard:TWO_PIN
- D4, D5, D6, D7: footprint Daughterboard:SOT-23-6_NoPad6 -> Package_TO_SOT_SMD:SOT-23-6
- U7: footprint Daughterboard:SOIC-28W_7.5x17.9mm_P1.27mm_NoPads11_14 -> Package_SO:SOIC-28W_7.5x17.9mm_P1.27mm
Connections:
- net +3V3_SW_LOGIC is gone; now on net +3V3_SW: C17.1, C18.1, C19.1, C20.1, C27.1, C28.1, J928.1 (PAD), R19.2, R20.2, R42.1, R43.1, R44.1, U5.8 (VDD), U6.1 (ADDR), U6.8 (VDD), U7.9 (VDD)
Changed lines of the file:
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@@
 	)
 	(symbol
-		(lib_id "Daughterboard:PWR_FLAG")
-		(at 408.94 237.49 0)
-		(unit 1)
-		(exclude_from_sim no)
-		(in_bom no)
-		(on_board no)
-		(dnp no)
-		(property "Reference" "#FLG7"
-			(at 405.13 226.06 0)
-			(effects (font (size 1.016 1.016)) (justify left))
-		)
-		(property "Value" "PWR_FLAG"
-			(at 405.13 228.6 0)
-			(effects (font (size 1.016 1.016)) (justify left))
-		)
-		(property "Footprint" ""
-			(at 408.94 237.49 0)
-			(effects (font (size 1.016 1.016)) (hide yes) (justify left))
-		)
-		(property "Datasheet" ""
-			(at 408.94 237.49 0)
-			(effects (font (size 1.016 1.016)) (hide yes) (justify left))
-		)
-		(property "Purchase Link" "https://www.digikey.com/en/products/result?keywords=PWR_FLAG"
-			(at 408.94 237.49 0)
-			(effects (font (size 1.016 1.016)) (hide yes) (justify left))
-		)
-		(instances
-			(project "Daughterboard"
-				(path "/d4b0641a-9c05-4a64-9f99-e24c4b75c101" (reference "#FLG7") (unit 1))
-			)
-		)
-	)
-	(wire (pts (xy 417.83 237.49) (xy 422.91 237.49)) (stroke (width 0) (type default)))
-	(wire (pts (xy 422.91 237.49) (xy 422.91 234.95)) (stroke (width 0) (type default)))
-	(global_label "+3V3_SW_LOGIC"
-		(shape bidirectional)
-		(at 422.91 234.95 0)
-		(fields_autoplaced yes)
-		(effects (font (size 0.889 0.889)))
-		(property "Intersheetrefs" "${INTERSHEET_REFS}" (at 422.91 234.95 0) (effects (font (size 0.889 0.889)) (hide yes)))
-	)
-	(symbol
 		(lib_id "Daughterboard:AP63200WU")
 		(at 91.44 264.16 0)
@@
 	(wire (pts (xy 487.68 54.61) (xy 492.76 54.61)) (stroke (width 0) (type default)))
 	(wire (pts (xy 492.76 54.61) (xy 492.76 52.07)) (stroke (width 0) (type default)))
-	(global_label "+3V3_SW_LOGIC"
+	(global_label "+3V3_SW"
 		(shape bidirectional)
 		(at 492.76 52.07 0)
@@
 	(wire (pts (xy 449.58 124.46) (xy 444.5 124.46)) (stroke (width 0) (type default)))
 	(wire (pts (xy 444.5 124.46) (xy 444.5 121.92)) (stroke (width 0) (type default)))
-	(global_label "+3V3_SW_LOGIC"
+	(global_label "+3V3_SW"
 		(shape bidirectional)
 		(at 444.5 121.92 0)
@@
 	(wire (pts (xy 487.68 127) (xy 492.76 127)) (stroke (width 0) (type default)))
 	(wire (pts (xy 492.76 127) (xy 492.76 124.46)) (stroke (width 0) (type default)))
-	(global_label "+3V3_SW_LOGIC"
+	(global_label "+3V3_SW"
 		(shape bidirectional)
 		(at 492.76 124.46 0)
@@
 	(symbol
 		(lib_id "Daughterboard:TWO_PIN")
-		(at 527.05 25.4 0)
-		(unit 1)
-		(exclude_from_sim no)
-		(in_bom yes)
-		(on_board yes)
-		(dnp no)
-		(property "Reference" "R45"
-			(at 521.97 12.7 0)
-			(effects (font (size 1.016 1.016)) (justify left))
-		)
-		(property "Value" "0R"
-			(at 521.97 15.24 0)
-			(effects (font (size 1.016 1.016)) (justify left))
-		)
-		(property "Footprint" "Resistor_SMD:R_0603_1608Metric"
-			(at 527.05 25.4 0)
-			(effects (font (size 1.016 1.016)) (hide yes) (justify left))
-		)
-		(property "Datasheet" ""
-			(at 527.05 25.4 0)
-			(effects (font (size 1.016 1.016)) (hide yes) (justify left))
-		)
-		(property "Purchase Link" "https://www.digikey.com/en/products/result?keywords=0R+Resistor_SMD%3AR_0603_1608Metric+resistor"
-			(at 527.05 25.4 0)
-			(effects (font (size 1.016 1.016)) (hide yes) (justify left))
-		)
-		(instances
-			(project "Daughterboard"
-				(path "/d4b0641a-9c05-4a64-9f99-e24c4b75c101" (reference "R45") (unit 1))
-			)
-		)
-	)
-	(wire (pts (xy 516.89 25.4) (xy 511.81 25.4)) (stroke (width 0) (type default)))
-	(wire (pts (xy 511.81 25.4) (xy 511.81 22.86)) (stroke (width 0) (type default)))
-	(global_label "+3V3_SW"
-		(shape bidirectional)
-		(at 511.81 22.86 0)
-		(fields_autoplaced yes)
-		(effects (font (size 0.889 0.889)))
-		(property "Intersheetrefs" "${INTERSHEET_REFS}" (at 511.81 22.86 0) (effects (font (size 0.889 0.889)) (hide yes)))
-	)
-	(wire (pts (xy 537.21 25.4) (xy 542.29 25.4)) (stroke (width 0) (type default)))
-	(wire (pts (xy 542.29 25.4) (xy 542.29 22.86)) (stroke (width 0) (type default)))
-	(global_label "+3V3_SW_LOGIC"
-		(shape bidirectional)
-		(at 542.29 22.86 0)
-		(fields_autoplaced yes)
-		(effects (font (size 0.889 0.889)))
-		(property "Intersheetrefs" "${INTERSHEET_REFS}" (at 542.29 22.86 0) (effects (font (size 0.889 0.889)) (hide yes)))
-	)
-	(symbol
-		(lib_id "Daughterboard:TWO_PIN")
 		(at 527.05 40.64 0)
 		(unit 1)
@@
 	(wire (pts (xy 537.21 40.64) (xy 542.29 40.64)) (stroke (width 0) (type default)))
 	(wire (pts (xy 542.29 40.64) (xy 542.29 38.1)) (stroke (width 0) (type default)))
-	(global_label "+3V3_SW_LOGIC"
+	(global_label "+3V3_SW"
 		(shape bidirectional)
 		(at 542.29 38.1 0)
@@
 	(wire (pts (xy 537.21 54.61) (xy 542.29 54.61)) (stroke (width 0) (type default)))
 	(wire (pts (xy 542.29 54.61) (xy 542.29 52.07)) (stroke (width 0) (type default)))
-	(global_label "+3V3_SW_LOGIC"
+	(global_label "+3V3_SW"
 		(shape bidirectional)
 		(at 542.29 52.07 0)
@@
 	(wire (pts (xy 516.89 74.93) (xy 511.81 74.93)) (stroke (width 0) (type default)))
 	(wire (pts (xy 511.81 74.93) (xy 511.81 72.39)) (stroke (width 0) (type default)))
-	(global_label "+3V3_SW_LOGIC"
+	(global_label "+3V3_SW"
 		(shape bidirectional)
 		(at 511.81 72.39 0)
@@
 	(wire (pts (xy 516.89 88.9) (xy 511.81 88.9)) (stroke (width 0) (type default)))
 	(wire (pts (xy 511.81 88.9) (xy 511.81 86.36)) (stroke (width 0) (type default)))
-	(global_label "+3V3_SW_LOGIC"
+	(global_label "+3V3_SW"
 		(shape bidirectional)
 		(at 511.81 86.36 0)
@@
 	(wire (pts (xy 516.89 146.05) (xy 511.81 146.05)) (stroke (width 0) (type default)))
 	(wire (pts (xy 511.81 146.05) (xy 511.81 143.51)) (stroke (width 0) (type default)))
-	(global_label "+3V3_SW_LOGIC"
+	(global_label "+3V3_SW"
 		(shape bidirectional)
 		(at 511.81 143.51 0)
@@
 	(wire (pts (xy 516.89 161.29) (xy 511.81 161.29)) (stroke (width 0) (type default)))
 	(wire (pts (xy 511.81 161.29) (xy 511.81 158.75)) (stroke (width 0) (type default)))
-	(global_label "+3V3_SW_LOGIC"
+	(global_label "+3V3_SW"
 		(shape bidirectional)
 		(at 511.81 158.75 0)
@@
 			(effects (font (size 1.016 1.016)) (justify left))
 		)
-		(property "Footprint" "Daughterboard:SOIC-28W_7.5x17.9mm_P1.27mm_NoPads11_14"
+		(property "Footprint" "Package_SO:SOIC-28W_7.5x17.9mm_P1.27mm"
 			(at 422.91 336.55 0)
 			(effects (font (size 1.016 1.016)) (hide yes) (justify left))
@@
 	)
 	(wire (pts (xy 422.91 389.89) (xy 422.91 384.81)) (stroke (width 0) (type default)))
-	(global_label "+3V3_SW_LOGIC"
+	(global_label "+3V3_SW"
 		(shape bidirectional)
 		(at 422.91 384.81 0)
@@
 	)
 	(wire (pts (xy 330.2 293.37) (xy 325.12 293.37)) (stroke (width 0) (type default)))
-	(global_label "+3V3_SW_LOGIC"
+	(global_label "+3V3_SW"
 		(shape bidirectional)
 		(at 325.12 293.37 0)
@@
 	)
 	(wire (pts (xy 330.2 308.61) (xy 325.12 308.61)) (stroke (width 0) (type default)))
-	(global_label "+3V3_SW_LOGIC"
+	(global_label "+3V3_SW"
 		(shape bidirectional)
 		(at 325.12 308.61 0)
@@
 	)
 	(wire (pts (xy 330.2 365.76) (xy 325.12 365.76)) (stroke (width 0) (type default)))
-	(global_label "+3V3_SW_LOGIC"
+	(global_label "+3V3_SW"
 		(shape bidirectional)
 		(at 325.12 365.76 0)
@@
 	)
 	(wire (pts (xy 421.64 293.37) (xy 416.56 293.37)) (stroke (width 0) (type default)))
-	(global_label "+3V3_SW_LOGIC"
+	(global_label "+3V3_SW"
 		(shape bidirectional)
 		(at 416.56 293.37 0)
@@
 	)
 	(wire (pts (xy 421.64 308.61) (xy 416.56 308.61)) (stroke (width 0) (type default)))
-	(global_label "+3V3_SW_LOGIC"
+	(global_label "+3V3_SW"
 		(shape bidirectional)
 		(at 416.56 308.61 0)
@@
 			(effects (font (size 1.016 1.016)) (justify left))
 		)
-		(property "Footprint" "Daughterboard:SOT-23-6_NoPad6"
+		(property "Footprint" "Package_TO_SOT_SMD:SOT-23-6"
 			(at 474.98 515.62 0)
 			(effects (font (size 1.016 1.016)) (hide yes) (justify left))
@@
 			(effects (font (size 1.016 1.016)) (justify left))
 		)
-		(property "Footprint" "Daughterboard:SOT-23-6_NoPad6"
+		(property "Footprint" "Package_TO_SOT_SMD:SOT-23-6"
 			(at 552.45 515.62 0)
 			(effects (font (size 1.016 1.016)) (hide yes) (justify left))
@@
 			(effects (font (size 1.016 1.016)) (justify left))
 		)
-		(property "Footprint" "Daughterboard:SOT-23-6_NoPad6"
+		(property "Footprint" "Package_TO_SOT_SMD:SOT-23-6"
 			(at 629.92 515.62 0)
 			(effects (font (size 1.016 1.016)) (hide yes) (justify left))
@@
 			(effects (font (size 1.016 1.016)) (justify left))
 		)
-		(property "Footprint" "Daughterboard:SOT-23-6_NoPad6"
+		(property "Footprint" "Package_TO_SOT_SMD:SOT-23-6"
 			(at 708.66 515.62 0)
 			(effects (font (size 1.016 1.016)) (hide yes) (justify left))
@@
 	)
 	(wire (pts (xy 769.62 482.6) (xy 774.7 482.6)) (stroke (width 0) (type default)))
-	(global_label "+3V3_SW_LOGIC"
+	(global_label "+3V3_SW"
 		(shape bidirectional)
 		(at 774.7 482.6 0)
