File: Daughterboard/Daughterboard_before_bom_netlist_cbset_eco.kicad_pcb (KiCad board)
At the start: 4 copper layers, 155 x 80.6 mm, 150 parts, among them J1 USB-C 5V Sink, J30 J3P Hosyond +5V_SW solder pad, J31 J3A Hosyond UART_TX solder pad, J32 J3B Hosyond UART_RX solder pad, J33 J3C Hosyond I2C_SDA solder pad, J34 J3D Hosyond I2C_SCL solder pad, J35 J3E Hosyond GPIO2 solder pad, J36 J3F Hosyond GPIO3 solder pad, J37 J3G Hosyond GPIO14 solder pad, J38 J3H Hosyond GPIO21 solder pad, J39 J3I Hosyond GND solder pad, J4 UART JST-GH 1.25mm, J5 I2C male header 2.54mm, J6 Deep sleep pushbutton header, J7 2S balance input JST-XH, J8 Analog input header, J91 MCP23017 GPA0 solder pad, J910 MCP23017 GPB1 solder pad, J911 MCP23017 GPB2 solder pad, J912 MCP23017 GPB3 solder pad, J913 MCP23017 GPB4 solder pad, J914 MCP23017 GPB5 solder pad, J915 MCP23017 GPB6 solder pad, J916 MCP23017 GPB7 solder pad, J92 MCP23017 GPA1 solder pad, J925 MCP23017 INTA solder pad, J926 MCP23017 INTB solder pad, J927 MCP23017 RESET solder pad, J928 MCP23017 +3V3_SW solder pad, J929 MCP23017 GND solder pad, J93 MCP23017 GPA2 solder pad, J94 MCP23017 GPA3 solder pad, J95 MCP23017 GPA4 solder pad, J96 MCP23017 GPA5 solder pad, J97 MCP23017 GPA6 solder pad, J98 MCP23017 GPA7 solder pad, J99 MCP23017 GPB0 solder pad, Q1 CSD83325L, SW1 Pololu #2808 5V switch, SW2 Pololu #2808 3V3 switch, U1 BQ25887RGE 2S charger, U2 S-8252AAH-M6T1U, U3 AP63200WU 5V Buck, U4 AP63200WU 3V3 Buck, U5 ADS1115IDGS 0x48, U6 ADS1115IDGS 0x49, U7 MCP23017-E/SO

Commit message: k
Parts:
- C8: value 100nF 10V X7R DNP -> 100nF 10V X7R
- D4, D5, D6, D7: value SP0504BAHTG 4ch GPIO TVS -> 4ch 3.3V GPIO TVS array TBD
- R3: value 806R 1% ILIM -> 806R 1% TBD
- R4: value 220R 1% CBSET -> TBD 1%
Connections:
- R4 pad 2: CELL_MID -> GND
Routing:
- net CELL_MID: track 62.0 -> 59.6 mm, vias 4 -> 3
- net GND: track 82.8 -> 84.0 mm, vias 47 -> 48
Changed lines of the file:
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@@
 			)
 		)
-		(property "Value" "806R 1% ILIM"
+		(property "Value" "806R 1% TBD"
 			(at 0 1.43 90)
 			(layer "F.Fab")
@@
 			)
 		)
-		(property "Value" "SP0504BAHTG 4ch GPIO TVS"
+		(property "Value" "4ch 3.3V GPIO TVS array TBD"
 			(at 0 2.4 0)
 			(layer "F.Fab")
@@
 			)
 		)
-		(property "Value" "100nF 10V X7R DNP"
+		(property "Value" "100nF 10V X7R"
 			(at 0 1.43 0)
 			(layer "F.Fab")
@@
 			)
 		)
-		(attr smd dnp)
+		(attr smd)
 		(duplicate_pad_numbers_are_jumpers no)
 		(fp_line
@@
 			)
 		)
-		(property "Value" "SP0504BAHTG 4ch GPIO TVS"
+		(property "Value" "4ch 3.3V GPIO TVS array TBD"
 			(at 0 2.4 0)
 			(layer "F.Fab")
@@
 			)
 		)
-		(property "Value" "SP0504BAHTG 4ch GPIO TVS"
+		(property "Value" "4ch 3.3V GPIO TVS array TBD"
 			(at 0 2.4 90)
 			(layer "F.Fab")
@@
 			)
 		)
-		(property "Value" "SP0504BAHTG 4ch GPIO TVS"
+		(property "Value" "4ch 3.3V GPIO TVS array TBD"
 			(at 0 2.4 0)
 			(layer "F.Fab")
@@
 			)
 		)
-		(property "Value" "220R 1% CBSET"
+		(property "Value" "TBD 1%"
 			(at 0 1.43 0)
 			(layer "F.Fab")
@@
 			(layers "F.Cu" "F.Mask" "F.Paste")
 			(roundrect_rratio 0.25)
-			(net "CELL_MID")
+			(net "GND")
 		)
 		(embedded_fonts no)
@@
 	)
 	(segment
+		(start 34 39.3)
+		(end 34.4841 38.8159)
+		(width 0.2)
+		(layer "F.Cu")
+		(net "GND")
+	)
+	(segment
 		(start 86.1606 16.6144)
 		(end 85.775 17)
@@
 	)
 	(segment
+		(start 34.4841 38.8159)
+		(end 34.9284 38.8159)
+		(width 0.2)
+		(layer "F.Cu")
+		(net "GND")
+	)
+	(segment
 		(start 159.9999 18.7)
 		(end 159.9999 19.9527)
@@
 	)
 	(via
+		(at 34.9284 38.8159)
+		(size 0.6)
+		(drill 0.3)
+		(layers "F.Cu" "B.Cu")
+		(net "GND")
+	)
+	(via
 		(at 140.7716 28.4618)
 		(size 0.6)
@@
 	)
 	(segment
-		(start 34.4841 38.8159)
-		(end 34.9284 38.8159)
-		(width 0.2)
-		(layer "F.Cu")
-		(net "CELL_MID")
-	)
-	(segment
 		(start 42.2 44.3081)
 		(end 44.2953 46.4034)
@@
 	)
 	(segment
-		(start 34 39.3)
-		(end 34.4841 38.8159)
-		(width 0.2)
-		(layer "F.Cu")
-		(net "CELL_MID")
-	)
-	(segment
 		(start 41.4 52.3767)
 		(end 41.4 57.8)
@@
 	)
 	(via
-		(at 34.9284 38.8159)
-		(size 0.6)
-		(drill 0.3)
-		(layers "F.Cu" "B.Cu")
-		(net "CELL_MID")
-	)
-	(via
 		(at 38.5324 44.2574)
 		(size 0.6)
@@
 		(width 0.2)
 		(layer "In2.Cu")
-		(net "CELL_MID")
-	)
-	(segment
-		(start 34.9284 38.8159)
-		(end 34 39.725)
-		(width 0.2)
-		(layer "In2.Cu")
