File: Daughterboard/Daughterboard_before_clear_traces.kicad_pcb (KiCad board)
At the start: 4 copper layers, 155 x 80.6 mm, 150 parts, among them J1 USB-C 5V Sink, J30 J3P Hosyond +5V_SW solder pad, J31 J3A Hosyond UART_TX solder pad, J32 J3B Hosyond UART_RX solder pad, J33 J3C Hosyond I2C_SDA solder pad, J34 J3D Hosyond I2C_SCL solder pad, J35 J3E Hosyond GPIO2 solder pad, J36 J3F Hosyond GPIO3 solder pad, J37 J3G Hosyond GPIO14 solder pad, J38 J3H Hosyond GPIO21 solder pad, J39 J3I Hosyond GND solder pad, J4 UART JST-GH 1.25mm, J5 I2C male header 2.54mm, J6 Deep sleep pushbutton header, J7 2S balance input JST-XH, J8 Analog input header, J91 MCP23017 GPA0 solder pad, J910 MCP23017 GPB1 solder pad, J911 MCP23017 GPB2 solder pad, J912 MCP23017 GPB3 solder pad, J913 MCP23017 GPB4 solder pad, J914 MCP23017 GPB5 solder pad, J915 MCP23017 GPB6 solder pad, J916 MCP23017 GPB7 solder pad, J92 MCP23017 GPA1 solder pad, J925 MCP23017 INTA solder pad, J926 MCP23017 INTB solder pad, J927 MCP23017 RESET solder pad, J928 MCP23017 +3V3_SW solder pad, J929 MCP23017 GND solder pad, J93 MCP23017 GPA2 solder pad, J94 MCP23017 GPA3 solder pad, J95 MCP23017 GPA4 solder pad, J96 MCP23017 GPA5 solder pad, J97 MCP23017 GPA6 solder pad, J98 MCP23017 GPA7 solder pad, J99 MCP23017 GPB0 solder pad, Q1 CSD83325L, SW1 Pololu #2808 5V switch, SW2 Pololu #2808 3V3 switch, U1 BQ25887RGE 2S charger, U2 S-8252AAH-M6T1U, U3 AP63200WU 5V Buck, U4 AP63200WU 3V3 Buck, U5 ADS1115IDGS 0x48, U6 ADS1115IDGS 0x49, U7 MCP23017-E/SO

Commit message: a
Routing:
- net DO_GATE: track 25.7 -> 0.00 mm
- net EN_3V3: track 18.8 -> 0.00 mm, vias 2 -> 0
- net BATT_RAW_N: track 91.9 -> 75.9 mm, vias 3 -> 1
- net GND: track 84.0 -> 74.9 mm
- net BTST: track 7.87 -> 0.00 mm, vias 2 -> 0
- net CHG_IN: track 35.6 -> 33.4 mm

Commit message: Update
Parts:
- removed TP13: VM_SENSE test pad, TestPoint_Pad_D1.0mm
- removed TP8: +5V_SW test pad, TestPoint_Pad_D1.0mm
- added C30: 2.2uF 10V X5R, C_0603_1608Metric, F.Cu at (70.8, 34.2)
- added C31: 100nF 16V X7R, C_0603_1608Metric, F.Cu at (71.8, 29.4)
- added R46: 2mR 1% 50ppm, R_1206_3216Metric, F.Cu at (55.0, 43.8)
- added R47: 100R, R_0603_1608Metric, F.Cu at (70.0, 24.0)
- added R48: 100R, R_0603_1608Metric, F.Cu at (72.2, 24.0)
- C13, C14, C22, C23: value 22uF 10V X5R -> 22uF 16V X5R
- C8: value 100nF 10V X7R -> 100nF 10V X7R DNP
- D4, D5, D6, D7: value 4ch 3.3V GPIO TVS array TBD -> SP0504BAHTG 4ch GPIO TVS
- J4: value UART JST-GH 1.25mm -> UART JST-GH top-entry 1.25mm; footprint JST_GH_SM05B-GHS-TB_1x05-1MP_P1.25mm_Horizontal -> JST_GH_BM05B-GHS-TBT_1x05-1MP_P1.25mm_Vertical
- R16: value 2.0k 1% -> 100R
- R3: value 806R 1% TBD -> 806R 1% ILIM
- R4: value TBD 1% -> 220R 1% CBSET
- U2: value S-8252AAH-M6T1U -> BQ28Z610DRZR-R1; footprint SOT-23-6 -> BQ28Z610_DRZ0012A_12SON_2.5x4mm_P0.5mm
- moved R14 1.40 mm to (90.0, 13.6), turned to 180 degrees
- turned J4 to 0 degrees
Connections:
- R16 pad 1: VM_SENSE -> BAT_SYS
- R16 pad 2: GND -> BQ_PACK
- R21 pad 1: S8252_DO -> BQ_DSG
- R22 pad 1: S8252_CO -> BQ_CHG
- R4 pad 2: GND -> CELL_MID
- U2 pad 1: S8252_DO -> BATT_RAW_N
- U2 pad 2: S8252_CO -> BQ_SRN
- U2 pad 3: VM_SENSE -> BQ_SRP
- U2 pad 4: PROT_VC -> TS
- U2 pad 5: PROT_VDD -> I2C_SCL
- U2 pad 6: BATT_RAW_N -> I2C_SDA
Routing:
- net I2C_SCL: track 186.6 -> 328.6 mm, vias 2 -> 3
- net I2C_SDA: track 178.9 -> 316.0 mm, vias 3 -> 4
- net TS: track 14.1 -> 111.1 mm
- net +3V3_SW: track 108.4 -> 195.3 mm
- net +3V3_SW_LOGIC: track 173.2 -> 256.6 mm
- net BAT_SYS: track 129.9 -> 210.3 mm, vias 4 -> 5
- net UART_RX: track 53.4 -> 130.8 mm
- net GPIO2: track 79.2 -> 147.6 mm, vias 3 -> 2
- net +5V: track 80.7 -> 148.4 mm
- net BATT_RAW_N: track 75.9 -> 142.1 mm, vias 1 -> 0
- net EXP_GPB7: track 69.8 -> 135.5 mm
- net USB_VBUS: track 69.8 -> 132.1 mm, vias 0 -> 2
- net +5V_SW: track 83.2 -> 143.3 mm, vias 1 -> 2
- net BQ_PACK: track 0.00 -> 55.0 mm
- net EXP_GPA5: track 34.3 -> 79.8 mm, vias 2 -> 0
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
Commit message: rep update
Parts:
- added J40: Left gimbal B JST-GH 1.25mm, JST_GH_BM03B-GHS-TBT_1x03-1MP_P1.25mm_Vertical, F.Cu at (33.0, 14.0)
- added J41: Right gimbal A JST-GH 1.25mm, JST_GH_BM03B-GHS-TBT_1x03-1MP_P1.25mm_Vertical, F.Cu at (139.0, 14.0)
- added J42: Right gimbal B JST-GH 1.25mm, JST_GH_BM03B-GHS-TBT_1x03-1MP_P1.25mm_Vertical, F.Cu at (151.0, 14.0)
- added TP15: AIN4 test pad, TestPoint_Pad_D1.0mm, F.Cu at (158.6, 13.3)
- added TP16: AIN5 test pad, TestPoint_Pad_D1.0mm, F.Cu at (162.4, 13.3)
- added TP17: AIN6 test pad, TestPoint_Pad_D1.0mm, F.Cu at (158.6, 16.6)
- added TP18: AIN7 test pad, TestPoint_Pad_D1.0mm, F.Cu at (162.4, 16.6)
- D1: value 5V VBUS TVS -> PESD5V0S1BA 5V VBUS TVS
- F1: value 2A hold polyfuse -> BSMD1206-200-16V 2A hold polyfuse
- F2: value PTC/fuse cell1 -> BSMD1206-200-16V cell1 PTC
- F3: value PTC/fuse cell2 -> BSMD1206-200-16V cell2 PTC
- F4: value 2A system fuse -> BSMD1206-200-16V system fuse
- J4: value UART JST-GH top-entry 1.25mm -> BM05B-GHS-TBT UART JST-GH top-entry 1.25mm
- J5: value I2C male header 2.54mm -> I2C SMD male header 2.54mm; footprint PinHeader_1x04_P2.54mm_Vertical -> PinHeader_1x04_P2.54mm_Vertical_SMD_Pin1Left
- J6: value Deep sleep pushbutton header -> Deep sleep SMD pushbutton header; footprint PinHeader_1x02_P2.54mm_Vertical -> PinHeader_1x02_P2.54mm_Vertical_SMD_Pin1Left
- J7: value 2S balance input JST-XH -> 2S balance input JST-XH side-entry; footprint JST_XH_B3B-XH-A_1x03_P2.50mm_Vertical -> JST_XH_S3B-XH-A_1x03_P2.50mm_Horizontal
- J8: value Analog input header -> Left gimbal A JST-GH 1.25mm; footprint PinHeader_1x10_P2.54mm_Vertical -> JST_GH_BM03B-GHS-TBT_1x03-1MP_P1.25mm_Vertical
- L3: value 1uH >=4A sat -> ANR5040T1R0M 1uH
- Q1: value CSD83325L -> PT8810 dual N-MOSFET; footprint CSD83325L_YJE0006A -> TSSOP-8_4.4x3mm_P0.65mm
- R4: value 220R 1% CBSET -> 43R 1W CBSET; footprint R_0603_1608Metric -> R_2512_6332Metric
- TH1: value 10k NTC -> NCP18XH103F03RB 10k NTC
- U1: value BQ25887RGE 2S charger -> BQ25887RGER 2S charger
- U3: value AP63200WU 5V Buck -> AP63200WU-7 5V Buck
- U4: value AP63200WU 3V3 Buck -> AP63200WU-7 3V3 Buck
- U5: value ADS1115IDGS 0x48 -> ADS1115IDGSR 0x48
- U6: value ADS1115IDGS 0x49 -> ADS1115IDGSR 0x49
- moved J8 116.8 mm to (21.0, 14.0), turned to 0 degrees
- moved U5 68.6 mm to (91.8, 23.7), turned to 180 degrees
- moved C16 61.9 mm to (31.7, 55.6), turned to 90 degrees
- moved D2 52.8 mm to (19.8, 75.3)
- moved D3 52.6 mm to (24.1, 75.4)
- moved C21 50.1 mm to (42.7, 43.9)
- moved J7 46.8 mm to (70.6, 16.5), turned to 180 degrees
- moved R14 44.9 mm to (53.5, 39.7), turned to -90 degrees
- moved D1 40.4 mm to (19.6, 71.7), turned to 180 degrees
- moved TP7 32.5 mm to (102.9, 33.6)
- moved C26 20.7 mm to (65.5, 22.0)
- moved C25 17.9 mm to (65.5, 25.5), turned to 180 degrees
- moved R4 13.9 mm to (42.0, 50.0)
- moved Q1 13.8 mm to (59.5, 50.0)
- moved R13 13.4 mm to (77.6, 24.0), turned to -90 degrees
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Connections:
- J8 pad 1: AIN0 -> GND
- J8 pad 2: AIN1 -> AIN0
- J8 pad 3: AIN2 -> +3V3_SW
Routing:
- net I2C_SCL: track 328.6 -> 109.5 mm, vias 3 -> 5
- net I2C_SDA: track 316.0 -> 118.1 mm
- net PACK_P: track 180.5 -> 51.2 mm, vias 2 -> 1
- net BAT_SYS: track 210.3 -> 101.8 mm, vias 5 -> 3
- net +3V3_SW_LOGIC: track 256.6 -> 160.2 mm, vias 3 -> 4
- net BATT_RAW_N: track 142.1 -> 52.0 mm
- net GPIO2: track 147.6 -> 61.2 mm, vias 2 -> 1
- net TS: track 111.1 -> 28.0 mm
- net +5V_SW: track 143.3 -> 69.8 mm, vias 2 -> 1
- net USB_VBUS: track 132.1 -> 64.8 mm, vias 2 -> 3
- net +5V: track 148.4 -> 82.6 mm
- net UART_RX: track 130.8 -> 65.9 mm
- net EXP_GPB7: track 135.5 -> 71.8 mm
- net +3V3_SW: track 195.3 -> 135.2 mm, vias 1 -> 3
- net EXP_GPB3: track 98.8 -> 42.2 mm, vias 3 -> 2
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Other:
- outline, holes or cut-outs redrawn
- board text added: "+5V_SW"
- board text added: "GND"
- board text added: "GPIO14"
- board text added: "GPIO2"
- board text added: "GPIO21"
- board text added: "GPIO3"
- board text added: "I2C_SCL"
- board text added: "I2C_SDA"
- board text added: "UART_RX"
- board text added: "UART_TX"
