File: Daughterboard/daughterboard.kicad_pcb (KiCad board)
At the start: 4 copper layers, 155 x 80.6 mm, 150 parts, among them J1 USB-C 5V Sink, J30 J3P Hosyond +5V_SW solder pad, J31 J3A Hosyond UART_TX solder pad, J32 J3B Hosyond UART_RX solder pad, J33 J3C Hosyond I2C_SDA solder pad, J34 J3D Hosyond I2C_SCL solder pad, J35 J3E Hosyond GPIO2 solder pad, J36 J3F Hosyond GPIO3 solder pad, J37 J3G Hosyond GPIO14 solder pad, J38 J3H Hosyond GPIO21 solder pad, J39 J3I Hosyond GND solder pad, J4 UART JST-GH 1.25mm, J5 I2C male header 2.54mm, J6 Deep sleep pushbutton header, J7 2S balance input JST-XH, J8 Analog input header, J91 MCP23017 GPA0 solder pad, J910 MCP23017 GPB1 solder pad, J911 MCP23017 GPB2 solder pad, J912 MCP23017 GPB3 solder pad, J913 MCP23017 GPB4 solder pad, J914 MCP23017 GPB5 solder pad, J915 MCP23017 GPB6 solder pad, J916 MCP23017 GPB7 solder pad, J92 MCP23017 GPA1 solder pad, J925 MCP23017 INTA solder pad, J926 MCP23017 INTB solder pad, J927 MCP23017 RESET solder pad, J928 MCP23017 +3V3_SW solder pad, J929 MCP23017 GND solder pad, J93 MCP23017 GPA2 solder pad, J94 MCP23017 GPA3 solder pad, J95 MCP23017 GPA4 solder pad, J96 MCP23017 GPA5 solder pad, J97 MCP23017 GPA6 solder pad, J98 MCP23017 GPA7 solder pad, J99 MCP23017 GPB0 solder pad, Q1 CSD83325L, SW1 Pololu #2808 5V switch, SW2 Pololu #2808 3V3 switch, U1 BQ25887RGE 2S charger, U2 S-8252AAH-M6T1U, U3 AP63200WU 5V Buck, U4 AP63200WU 3V3 Buck, U5 ADS1115IDGS 0x48, U6 ADS1115IDGS 0x49, U7 MCP23017-E/SO

Commit message: Update
Parts:
- removed TP13: VM_SENSE test pad, TestPoint_Pad_D1.0mm
- removed TP8: +5V_SW test pad, TestPoint_Pad_D1.0mm
- added C30: 2.2uF 10V X5R, C_0603_1608Metric, F.Cu at (70.8, 34.2)
- added C31: 100nF 16V X7R, C_0603_1608Metric, F.Cu at (71.8, 29.4)
- added J40: Left gimbal B JST-GH 1.25mm, JST_GH_BM03B-GHS-TBT_1x03-1MP_P1.25mm_Vertical, F.Cu at (33.0, 14.0)
- added J41: Right gimbal A JST-GH 1.25mm, JST_GH_BM03B-GHS-TBT_1x03-1MP_P1.25mm_Vertical, F.Cu at (139.0, 14.0)
- added J42: Right gimbal B JST-GH 1.25mm, JST_GH_BM03B-GHS-TBT_1x03-1MP_P1.25mm_Vertical, F.Cu at (151.0, 14.0)
- added R46: 2mR 1% 50ppm, R_1206_3216Metric, F.Cu at (53.9, 46.3)
- added R47: 100R, R_0603_1608Metric, F.Cu at (70.0, 24.0)
- added R48: 100R, R_0603_1608Metric, F.Cu at (73.8, 24.0)
- added TP15: AIN4 test pad, TestPoint_Pad_D1.0mm, F.Cu at (158.6, 13.3)
- added TP16: AIN5 test pad, TestPoint_Pad_D1.0mm, F.Cu at (162.4, 13.3)
- added TP17: AIN6 test pad, TestPoint_Pad_D1.0mm, F.Cu at (158.6, 16.6)
- added TP18: AIN7 test pad, TestPoint_Pad_D1.0mm, F.Cu at (162.4, 16.6)
- C13, C14, C22, C23: value 22uF 10V X5R -> 22uF 16V X5R
- J4: value UART JST-GH 1.25mm -> UART JST-GH top-entry 1.25mm; footprint JST_GH_SM05B-GHS-TB_1x05-1MP_P1.25mm_Horizontal -> JST_GH_BM05B-GHS-TBT_1x05-1MP_P1.25mm_Vertical
- J7: value 2S balance input JST-XH -> 2S balance input JST-XH side-entry; footprint JST_XH_B3B-XH-A_1x03_P2.50mm_Vertical -> JST_XH_S3B-XH-A_1x03_P2.50mm_Horizontal
- J8: value Analog input header -> Left gimbal A JST-GH 1.25mm; footprint PinHeader_1x10_P2.54mm_Vertical -> JST_GH_BM03B-GHS-TBT_1x03-1MP_P1.25mm_Vertical
- R16: value 2.0k 1% -> 100R
- U2: value S-8252AAH-M6T1U -> BQ28Z610DRZR-R1; footprint SOT-23-6 -> BQ28Z610_DRZ0012A_12SON_2.5x4mm_P0.5mm
- moved J8 116.8 mm to (21.0, 14.0), turned to 0 degrees
- moved U5 68.6 mm to (91.8, 23.7), turned to 180 degrees
- moved C16 61.9 mm to (31.7, 55.6), turned to 90 degrees
- moved D2 52.8 mm to (19.8, 75.3)
- moved D3 52.6 mm to (24.1, 75.4)
- moved C21 50.1 mm to (42.7, 43.9)
- moved J7 46.8 mm to (70.6, 16.5), turned to 180 degrees
- moved R14 44.1 mm to (53.5, 39.7), turned to -90 degrees
- moved D1 40.4 mm to (19.6, 71.7), turned to 180 degrees
- moved TP7 32.5 mm to (102.9, 33.6)
- moved C26 20.7 mm to (65.5, 22.0)
- moved C25 17.9 mm to (65.5, 25.5), turned to 180 degrees
- moved R13 13.4 mm to (77.6, 24.0), turned to -90 degrees
- moved C10 11.7 mm to (52.4, 36.1)
- moved C24 10.4 mm to (89.9, 19.4)
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Connections:
- J8 pad 1: AIN0 -> GND
- J8 pad 2: AIN1 -> AIN0
- J8 pad 3: AIN2 -> +3V3_SW
- R16 pad 1: VM_SENSE -> BAT_SYS
- R16 pad 2: GND -> BQ_PACK
- R21 pad 1: S8252_DO -> BQ_DSG
- R22 pad 1: S8252_CO -> BQ_CHG
- U2 pad 1: S8252_DO -> BATT_RAW_N
- U2 pad 2: S8252_CO -> BQ_SRN
- U2 pad 3: VM_SENSE -> BQ_SRP
- U2 pad 4: PROT_VC -> TS
- U2 pad 5: PROT_VDD -> I2C_SCL
- U2 pad 6: BATT_RAW_N -> I2C_SDA
Routing:
- net LED_CHG_A: track 3.86 -> 64.7 mm, vias 0 -> 2
- net +3V3_SW: track 108.4 -> 163.7 mm, vias 1 -> 3
- net PACK_P: track 135.7 -> 84.2 mm, vias 2 -> 3
- net TS: track 14.1 -> 62.0 mm, vias 3 -> 4
- net AIN0: track 32.9 -> 80.5 mm, vias 1 -> 2
- net LED_PGOOD_A: track 7.12 -> 53.3 mm, vias 0 -> 2
- net VM_SENSE: track 45.0 -> 0.00 mm, vias 3 -> 0
- net AIN3: track 22.7 -> 66.3 mm, vias 1 -> 2
- net PG_STAT: track 39.6 -> 82.9 mm, vias 2 -> 4
- net CHG_STAT: track 42.0 -> 78.6 mm, vias 2 -> 3
- net CHG_IN: track 35.6 -> 71.1 mm, vias 0 -> 2
- net AIN1: track 32.8 -> 64.2 mm, vias 1 -> 2
- net +3V3_SW_LOGIC: track 173.2 -> 204.2 mm, vias 3 -> 4
- net BATT_RAW_N: track 91.9 -> 62.9 mm, vias 3 -> 0
- net AIN2: track 27.6 -> 55.5 mm, vias 1 -> 2
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Other:
- board text added: "+5V_SW"
- board text added: "GND"
- board text added: "GPIO14"
- board text added: "GPIO2"
- board text added: "GPIO21"
- board text added: "GPIO3"
- board text added: "I2C_SCL"
- board text added: "I2C_SDA"
- board text added: "UART_RX"
- board text added: "UART_TX"

Commit message: a
Routing:
- net BATT_RAW_N: track 62.9 -> 72.5 mm, vias 0 -> 2
- net GND: track 76.4 -> 83.9 mm
- net DO_GATE: track 25.3 -> 27.8 mm
Changed lines of the file:
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@@
 	)
 	(gr_line
+		(start 47.9 44.6)
+		(end 46.6 44.6)
+		(stroke
+			(width 0.2)
+			(type default)
+		)
+		(layer "F.Cu")
+		(net "BATT_RAW_N")
+	)
+	(gr_line
 		(start 10 10.36904)
 		(end 61.470425 10.36904)
@@
 	)
 	(segment
+		(start 39.056 39.1073)
+		(end 44.2676 44.3189)
+		(width 0.2)
+		(layer "B.Cu")
+		(net "GND")
+	)
+	(segment
+		(start 44.2676 44.3189)
+		(end 44.4528 44.3189)
+		(width 0.2)
+		(layer "B.Cu")
+		(net "GND")
+	)
+	(segment
 		(start 151.7982 56.5982)
 		(end 151.7982 62.9501)
@@
 	)
 	(segment
+		(start 46.6 48.3)
+		(end 48.1 48.3)
+		(width 1)
+		(layer "F.Cu")
+		(net "BATT_RAW_N")
+	)
+	(segment
 		(start 64.6625 29.6311)
 		(end 69.4686 24.825)
@@
 	)
 	(segment
+		(start 51.25 45.15)
+		(end 50.7301 44.6301)
+		(width 1)
+		(layer "F.Cu")
+		(net "BATT_RAW_N")
+	)
+	(segment
 		(start 65.9784 33.425)
 		(end 70.8 33.425)
@@
 	(segment
 		(start 52.4 46.3)
-		(end 50.7301 44.6301)
+		(end 51.25 45.15)
 		(width 1)
 		(layer "F.Cu")
@@
 	)
 	(segment
+		(start 48.1 48.3)
+		(end 51.25 45.15)
+		(width 1)
+		(layer "F.Cu")
+		(net "BATT_RAW_N")
+	)
+	(segment
 		(start 59.8843 36.1)
 		(end 62.1612 36.1)
@@
 		(net "BATT_RAW_N")
 	)
+	(via
+		(at 46.6 48.3)
+		(size 0.6)
+		(drill 0.3)
+		(layers "F.Cu" "B.Cu")
+		(net "BATT_RAW_N")
+	)
+	(via
+		(at 46.6 44.6)
+		(size 0.6)
+		(drill 0.3)
+		(layers "F.Cu" "B.Cu")
+		(net "BATT_RAW_N")
+	)
+	(segment
+		(start 46.6 44.6)
+		(end 46.6 48.3)
+		(width 1)
+		(layer "In1.Cu")
+		(net "BATT_RAW_N")
+	)
 	(segment
 		(start 144.749 27.0176)
@@
 	)
 	(segment
-		(start 48.55 44.6596)
-		(end 48.1079 45.1017)
+		(start 45.95 44.869239)
+		(end 45.95 44.330761)
 		(width 0.2)
 		(layer "F.Cu")
@@
 	)
 	(segment
-		(start 48.1079 45.1017)
-		(end 47.6517 45.1017)
+		(start 64.9943 35.5407)
+		(end 65.5407 35.5407)
 		(width 0.2)
 		(layer "F.Cu")
@@
 	)
 	(segment
-		(start 47.3102 44.7602)
-		(end 47.3102 43.0089)
+		(start 45.95 44.330761)
+		(end 47.680761 42.6)
 		(width 0.2)
 		(layer "F.Cu")
@@
 	)
 	(segment
-		(start 64.9943 35.5407)
-		(end 65.5407 35.5407)
+		(start 48.2 42.6)
+		(end 48.2 42.1191)
 		(width 0.2)
 		(layer "F.Cu")
@@
 	)
 	(segment
-		(start 47.3102 43.0089)
-		(end 48.2335 42.0856)
+		(start 47.680761 42.6)
+		(end 48.2 42.6)
 		(width 0.2)
 		(layer "F.Cu")
@@
 	)
 	(segment
-		(start 47.6517 45.1017)
-		(end 47.3102 44.7602)
+		(start 48.55 44.6)
+		(end 48.55 44.6596)
+		(width 0.2)
+		(layer "F.Cu")
+		(net "DO_GATE")
+	)
+	(segment
+		(start 46.330761 45.25)
+		(end 45.95 44.869239)
 		(width 0.2)
 		(layer "F.Cu")
@@
 	)
 	(segment
-		(start 48.55 44.6)
-		(end 48.55 44.6596)
+		(start 48.55 44.6596)
+		(end 47.9596 45.25)
+		(width 0.2)
+		(layer "F.Cu")
+		(net "DO_GATE")
+	)
+	(segment
+		(start 47.9596 45.25)
+		(end 46.330761 45.25)
+		(width 0.2)
+		(layer "F.Cu")
+		(net "DO_GATE")
+	)
+	(segment
+		(start 48.2 42.1191)
+		(end 48.2335 42.0856)
 		(width 0.2)
 		(layer "F.Cu")
@@
 	(zone
 		(net "GND")
+		(locked yes)
 		(layer "In1.Cu")
 		(hatch edge 0.5)

Commit message: rep update
Parts:
- D1: value 5V VBUS TVS -> PESD5V0S1BA 5V VBUS TVS
- D4, D5, D6, D7: value SP0504BAHTG 4ch GPIO TVS -> SRV05-4.TCT / C13612 4ch ESD; footprint SOT-23-6_NoPad6 -> SOT-23-6
- F1: value 2A hold polyfuse -> BSMD1206-200-16V 2A hold polyfuse
- F2: value PTC/fuse cell1 -> BSMD1206-200-16V cell1 PTC
- F3: value PTC/fuse cell2 -> BSMD1206-200-16V cell2 PTC
- F4: value 2A system fuse -> BSMD1206-200-16V system fuse
- J4: value UART JST-GH top-entry 1.25mm -> BM05B-GHS-TBT UART JST-GH top-entry 1.25mm
- J5: value I2C male header 2.54mm -> I2C 2.54mm through-hole male header
- J6: value Deep sleep pushbutton header -> Deep sleep 2.54mm through-hole header
- L3: value 1uH >=4A sat -> ANR5040T1R0M 1uH
- Q1: value CSD83325L -> PT8810 dual N-MOSFET; footprint CSD83325L_YJE0006A -> TSSOP-8_4.4x3mm_P0.65mm
- R4: value 220R 1% CBSET -> 43R 1W CBSET; footprint R_0603_1608Metric -> R_2512_6332Metric
- TH1: value 10k NTC -> NCP18XH103F03RB 10k NTC
- U1: value BQ25887RGE 2S charger -> BQ25887RGER 2S charger
- U3: value AP63200WU 5V Buck -> AP63200WU-7 5V Buck
- U4: value AP63200WU 3V3 Buck -> AP63200WU-7 3V3 Buck
- U5: value ADS1115IDGS 0x48 -> ADS1115IDGSR 0x48
- U6: value ADS1115IDGS 0x49 -> ADS1115IDGSR 0x49
- moved R4 13.9 mm to (42.0, 50.0)
- moved Q1 12.4 mm to (59.5, 50.0)
Connections:
- D4 pad 2: EXP_GPA1 -> GND
- D4 pad 3: GND -> EXP_GPA1
- D4 pad 5: EXP_GPA3 -> +3V3_SW_LOGIC
- D5 pad 2: EXP_GPA5 -> GND
- D5 pad 3: GND -> EXP_GPA5
- D5 pad 5: EXP_GPA7 -> +3V3_SW_LOGIC
- D6 pad 2: EXP_GPB1 -> GND
- D6 pad 3: GND -> EXP_GPB1
- D6 pad 5: EXP_GPB3 -> +3V3_SW_LOGIC
- D7 pad 2: EXP_GPB5 -> GND
- D7 pad 3: GND -> EXP_GPB5
- D7 pad 5: EXP_GPB7 -> +3V3_SW_LOGIC
Routing:
- net +3V3_SW_LOGIC: track 204.2 -> 237.0 mm, vias 4 -> 8
- net CELL_MID: track 85.7 -> 103.6 mm
- net CO_GATE: track 3.17 -> 19.2 mm
- net I2C_SCL: track 180.9 -> 194.5 mm, vias 5 -> 6
- net CBSET: track 12.2 -> 25.6 mm
- net BQ_PACK: track 24.4 -> 37.4 mm
- net CHG_STAT: track 78.6 -> 91.6 mm
- net EXP_GPB2: track 32.2 -> 42.5 mm, vias 2 -> 3
- net +3V3_SW: track 163.7 -> 173.1 mm, vias 3 -> 4
- net +5V_SW: track 69.8 -> 78.5 mm
- net USB_VBUS: track 88.7 -> 80.1 mm
- net I2C_SDA: track 187.8 -> 180.3 mm, vias 5 -> 6
- net PROT_VDD: track 30.7 -> 23.8 mm, vias 2 -> 3
- net MCP_GPA1: track 24.0 -> 31.0 mm
- net MCP_GPA3: track 23.0 -> 29.8 mm
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Other:
- outline, holes or cut-outs redrawn

Commit message: R14
Parts:
- added C32: 100nF 25V X7R, C_0603_1608Metric, F.Cu at (38.5, 48.6)
- added C33: 100nF 25V X7R, C_0603_1608Metric, F.Cu at (22.8, 29.9)
- added Q2: CSD18502Q5B discharge FET, CSD18502Q5B_DNK0008A_VSON-CLIP_5x6mm, F.Cu at (17.3, 29.5)
- added R49: 10M, R_0603_1608Metric, F.Cu at (12.4, 29.4)
- added R50: 10M, R_0603_1608Metric, F.Cu at (28.1, 48.6)
- added TP13: BATT_RAW_P test pad, TestPoint_Pad_D1.0mm, F.Cu at (61.9, 52.5)
- Q1: value PT8810 dual N-MOSFET -> CSD18502Q5B charge FET; footprint TSSOP-8_4.4x3mm_P0.65mm -> CSD18502Q5B_DNK0008A_VSON-CLIP_5x6mm
- TP3: value PACK_P test pad -> BAT_SYS test pad
- moved Q1 26.8 mm to (32.7, 48.5), turned to 0 degrees
- moved TP1 12.8 mm to (20.8, 51.9)
- moved TH1 6.83 mm to (33.6, 40.8)
- moved R4 5.96 mm to (47.7, 51.6)
- moved R17 5.12 mm to (48.2, 47.2)
- moved TP2 0.60 mm to (24.8, 39.8)
- moved TP3 0.60 mm to (24.8, 43.6)
- moved TP5 0.60 mm to (24.8, 47.6)
Connections:
- C5 pad 1: PACK_P -> BAT_SYS
- C9 pad 1: PACK_P -> BATT_RAW_P
- F3 pad 2: PACK_P -> BATT_RAW_P
- F4 pad 1: PACK_P -> FET_BATT_P
- F4 pad 2: BAT_SYS -> BATT_RAW_P
- J7 pad 3: PACK_P -> BATT_RAW_P
- Q1 pad 1: BATT_RAW_N -> FET_SRC_COMMON
- Q1 pad 2: DO_GATE -> FET_SRC_COMMON
- Q1 pad 3: GND -> FET_SRC_COMMON
- Q1 pad 5: Q1_DRAIN_COMMON -> BAT_SYS
- Q1 pad 6: Q1_DRAIN_COMMON -> BAT_SYS
- Q1 pad 7: Q1_DRAIN_COMMON -> BAT_SYS
- Q1 pad 8: Q1_DRAIN_COMMON -> BAT_SYS
- R14 pad 1: PACK_P -> BATT_RAW_P
- R47 pad 1: BATT_RAW_N -> GND
- R48 pad 1: GND -> BATT_RAW_N
- TP3 pad 1: PACK_P -> BAT_SYS
- U1 pad 13: PACK_P -> BAT_SYS
- U1 pad 14: PACK_P -> BAT_SYS
- U1 pad 15: PACK_P -> BAT_SYS
- U1 pad 16: PACK_P -> BAT_SYS
Routing:
- net BATT_RAW_P: track 0.00 -> 90.9 mm, vias 0 -> 3
- net PACK_P: track 86.4 -> 0.00 mm, vias 2 -> 0
- net FET_SRC_COMMON: track 0.00 -> 51.6 mm, vias 0 -> 3
- net DO_GATE: track 22.0 -> 57.6 mm
- net BAT_SYS: track 104.6 -> 136.7 mm, vias 2 -> 5
- net FET_BATT_P: track 0.00 -> 26.7 mm
- net PROT_VDD: track 23.8 -> 41.6 mm, vias 3 -> 2
- net CHG_IN: track 70.6 -> 87.9 mm, vias 2 -> 3
- net +3V3_SW_LOGIC: track 237.0 -> 224.4 mm, vias 8 -> 2
- net BQ_PACK: track 37.4 -> 26.0 mm, vias 2 -> 0
- net CBSET: track 25.6 -> 36.5 mm
- net BATT_RAW_N: track 75.2 -> 65.3 mm, vias 2 -> 0
- net EXP_GPB2: track 42.5 -> 33.7 mm
- net LED_CHG_A: track 71.3 -> 62.8 mm
- net CHG_STAT: track 91.6 -> 83.2 mm
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