File: Daughterboard/daughterboard.kicad_sch (KiCad schematic)
At the start: 153 parts, among them J1 USB-C 5V Sink, J2 Switched power outputs, J30 J3P Hosyond +5V_SW solder pad, J31 J3A Hosyond UART_TX solder pad, J32 J3B Hosyond UART_RX solder pad, J33 J3C Hosyond I2C_SDA solder pad, J34 J3D Hosyond I2C_SCL solder pad, J35 J3E Hosyond GPIO2 solder pad, J36 J3F Hosyond GPIO3 solder pad, J37 J3G Hosyond GPIO14 solder pad, J38 J3H Hosyond GPIO21 solder pad, J39 J3I Hosyond GND solder pad, J4 UART JST-GH 1.25mm, J5 I2C male header 2.54mm, J6 Deep sleep pushbutton header, J7 2S balance input JST-XH, J8 Analog input header, J91 MCP23017 GPA0 solder pad, J910 MCP23017 GPB1 solder pad, J911 MCP23017 GPB2 solder pad, J912 MCP23017 GPB3 solder pad, J913 MCP23017 GPB4 solder pad, J914 MCP23017 GPB5 solder pad, J915 MCP23017 GPB6 solder pad, J916 MCP23017 GPB7 solder pad, J92 MCP23017 GPA1 solder pad, J925 MCP23017 INTA solder pad, J926 MCP23017 INTB solder pad, J927 MCP23017 RESET solder pad, J928 MCP23017 +3V3_SW solder pad, J929 MCP23017 GND solder pad, J93 MCP23017 GPA2 solder pad, J94 MCP23017 GPA3 solder pad, J95 MCP23017 GPA4 solder pad, J96 MCP23017 GPA5 solder pad, J97 MCP23017 GPA6 solder pad, J98 MCP23017 GPA7 solder pad, J99 MCP23017 GPB0 solder pad, Q1 CSD83325L, SW1 Pololu #2808 5V switch, SW2 Pololu #2808 3V3 switch, U1 BQ25887RGE 2S charger, U2 S-8252AAH-M6T1U, U3 AP63200WU 5V Buck, U4 AP63200WU 3V3 Buck, U5 ADS1115IDGS 0x48, U6 ADS1115IDGS 0x49, U7 MCP23017-E/SO

Commit message: Update
Parts:
- removed J8: Analog input header, Connector_PinHeader_2.54mm:PinHeader_1x10_P2.54mm_Vertical, symbol Daughterboard:CONN_10
- removed TP13: VM_SENSE test pad, TestPoint:TestPoint_Pad_D1.0mm, symbol Daughterboard:TESTPAD
- removed U2: S-8252AAH-M6T1U, Package_TO_SOT_SMD:SOT-23-6, symbol Daughterboard:S8252A_M6
- added C30: 2.2uF 10V X5R, Capacitor_SMD:C_0603_1608Metric, symbol Daughterboard:TWO_PIN
- added C31: 100nF 16V X7R, Capacitor_SMD:C_0603_1608Metric, symbol Daughterboard:TWO_PIN
- added J40: Left gimbal B JST-GH 1.25mm, Connector_JST:JST_GH_BM03B-GHS-TBT_1x03-1MP_P1.25mm_Vertical, symbol Daughterboard:CONN_3
- added J41: Right gimbal A JST-GH 1.25mm, Connector_JST:JST_GH_BM03B-GHS-TBT_1x03-1MP_P1.25mm_Vertical, symbol Daughterboard:CONN_3
- added J42: Right gimbal B JST-GH 1.25mm, Connector_JST:JST_GH_BM03B-GHS-TBT_1x03-1MP_P1.25mm_Vertical, symbol Daughterboard:CONN_3
- added J8: Left gimbal A JST-GH 1.25mm, Connector_JST:JST_GH_BM03B-GHS-TBT_1x03-1MP_P1.25mm_Vertical, symbol Daughterboard:CONN_3
- added R46: 2mR 1% 50ppm, Resistor_SMD:R_1206_3216Metric, symbol Daughterboard:TWO_PIN
- added R47, R48: 100R, Resistor_SMD:R_0603_1608Metric, symbol Daughterboard:TWO_PIN
- added TP15: AIN4 test pad, TestPoint:TestPoint_Pad_D1.0mm, symbol Daughterboard:TESTPAD
- added TP16: AIN5 test pad, TestPoint:TestPoint_Pad_D1.0mm, symbol Daughterboard:TESTPAD
- added TP17: AIN6 test pad, TestPoint:TestPoint_Pad_D1.0mm, symbol Daughterboard:TESTPAD
- added TP18: AIN7 test pad, TestPoint:TestPoint_Pad_D1.0mm, symbol Daughterboard:TESTPAD
- added U2: BQ28Z610DRZR-R1, Daughterboard:BQ28Z610_DRZ0012A_12SON_2.5x4mm_P0.5mm, symbol Daughterboard:BQ28Z610_DRZ
- C17: value 100nF 10V X7R DNP -> 100nF 10V X7R
- C8: now fitted
- D4, D5, D6, D7: value SP0504BAHTG 4ch GPIO TVS -> 4ch 3.3V GPIO TVS array TBD; Purchase Link https://www.digikey.com/en/products/result?keywords=SP0504B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 -> https://www.digikey.com/en/products/result?keywords=4+chann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
- J7: value 2S balance input JST-XH -> 2S balance input JST-XH side-entry; footprint Connector_JST:JST_XH_B3B-XH-A_1x03_P2.50mm_Vertical -> Connector_JST:JST_XH_S3B-XH-A_1x03_P2.50mm_Horizontal; Purchase Link https://www.digikey.com/en/products/result?keywords=JST+XH+3+pin+vertical+B3B-XH-A -> https://www.digikey.com/en/products/result?keywords=JST+XH+3+pin+horizontal+S3B-XH-A
- J928: value MCP23017 +3V3_SW solder pad -> MCP23017 +3V3_SW_LOGIC solder pad
- R16: value 2.0k 1% -> 100R; Purchase Link https://www.digikey.com/en/products/result?keywords=2.0k+1%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 -> https://www.digikey.com/en/products/result?keywords=100R+Re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
- R3: value 806R 1% ILIM -> 806R 1% TBD; Purchase Link https://www.digikey.com/en/products/result?keywords=806+ohm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 -> https://www.digikey.com/en/products/result?keywords=0603+re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
- R4: value 220R 1% CBSET -> TBD 1%; Purchase Link https://www.digikey.com/en/products/result?keywords=220+ohm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 -> https://www.digikey.com/en/products/result?keywords=0603+re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
Connections:
- net VM_SENSE is gone; now on net BAT_SYS: R16.1
- net +3V3_SW: now also J40.3, J41.3, J42.3, J8.3
- net AIN0: now also J8.2
- net AIN1: now also J40.2
- net AIN2: now also J41.2
- net AIN3: now also J42.2
- net AIN4: now also TP15.1 (PAD)
- net AIN5: now also TP16.1 (PAD)
- net AIN6: now also TP17.1 (PAD)
- net AIN7: now also TP18.1 (PAD)
- net BATT_RAW_N: now also C30.2, R46.1, R47.1, U2.1 (VSS), U2.13 (PWPD)
- net CELL_MID: no longer R4.2
- net GND: now also R4.2, J40.1, J41.1, J42.1, J8.1, R46.2, R48.1; no longer R16.2
- net I2C_SCL: now also U2.5 (SCL)
- net I2C_SDA: now also U2.6 (SDA)
- net PROT_VC: now also U2.12 (VC1)
- net PROT_VDD: now also U2.11 (VC2)
- net TS: now also U2.4 (TS1)
- net S8252_CO renamed BQ_CHG
- net BQ_CHG: now also U2.9 (CHG)
- net S8252_DO renamed BQ_DSG
- net BQ_DSG: now also U2.7 (DSG)
- new net BQ_PACK: R16.2, U2.8 (PACK)
- new net BQ_PBI: C30.1, U2.10 (PBI)
- new net BQ_SRN: C31.1, R47.2, U2.2 (SRN)
- new net BQ_SRP: C31.2, R48.2, U2.3 (SRP)

Commit message: rep update
Parts:
- D1: value 5V VBUS TVS -> PESD5V0S1BA 5V VBUS TVS
- D4, D5, D6, D7: value 4ch 3.3V GPIO TVS array TBD -> SRV05-4.TCT / C13612 4ch ESD; footprint Daughterboard:SOT-23-6_NoPad6 -> Package_TO_SOT_SMD:SOT-23-6; Purchase Link https://www.digikey.com/en/products/result?keywords=4+chann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 -> https://jlcpcb.com/partdetail/Semtech-SRV05_4TCT/C13612
- F1: value 2A hold polyfuse -> BSMD1206-200-16V 2A hold polyfuse
- F2: value PTC/fuse cell1 -> BSMD1206-200-16V cell1 PTC
- F3: value PTC/fuse cell2 -> BSMD1206-200-16V cell2 PTC
- F4: value 2A system fuse -> BSMD1206-200-16V system fuse
- J4: value UART JST-GH 1.25mm -> BM05B-GHS-TBT UART JST-GH top-entry 1.25mm; footprint Connector_JST:JST_GH_SM05B-GHS-TB_1x05-1MP_P1.25mm_Horizontal -> Connector_JST:JST_GH_BM05B-GHS-TBT_1x05-1MP_P1.25mm_Vertical; Purchase Link https://www.digikey.com/en/products/result?keywords=SM05B-G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 -> https://jlcpcb.com/partdetail/JST-BM05BGHSTBTLF_SN_N/C189891
- J5: value I2C male header 2.54mm -> I2C 2.54mm through-hole male header; Purchase Link https://www.digikey.com/en/products/result?keywords=2.54mm+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 -> (none)
- J6: value Deep sleep pushbutton header -> Deep sleep 2.54mm through-hole header; Purchase Link https://www.digikey.com/en/products/result?keywords=2.54mm+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 -> (none)
- L3: value 1uH >=4A sat -> ANR5040T1R0M 1uH
- Q1: value CSD83325L -> PT8810 dual N-MOSFET; footprint Daughterboard:CSD83325L_YJE0006A -> Package_SO:TSSOP-8_4.4x3mm_P0.65mm; symbol Daughterboard:PROT_FET_PAIR -> Daughterboard:PT8810_TSSOP8; Purchase Link https://www.digikey.com/en/products/result?keywords=CSD8332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 -> https://jlcpcb.com/partdetail/PT-PT8810/C3019811
- R3: Purchase Link https://www.digikey.com/en/products/result?keywords=0603+re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 -> https://jlcpcb.com/partdetail/C2692785
- R4: value TBD 1% -> 43R 1W CBSET; footprint Resistor_SMD:R_0603_1608Metric -> Resistor_SMD:R_2512_6332Metric; Purchase Link https://www.digikey.com/en/products/result?keywords=0603+re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 -> https://jlcpcb.com/partdetail/C38957
- TH1: value 10k NTC -> NCP18XH103F03RB 10k NTC
- U1: value BQ25887RGE 2S charger -> BQ25887RGER 2S charger; Purchase Link https://www.digikey.com/en/products/result?keywords=BQ25887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 -> https://jlcpcb.com/partdetail/TexasInstruments-BQ25887RGER/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
- U3: value AP63200WU 5V Buck -> AP63200WU-7 5V Buck; Purchase Link https://www.digikey.com/en/products/result?keywords=AP63200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 -> https://jlcpcb.com/partdetail/DiodesIncorporated-AP63200WU7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
- U4: value AP63200WU 3V3 Buck -> AP63200WU-7 3V3 Buck; Purchase Link https://www.digikey.com/en/products/result?keywords=AP63200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 -> https://jlcpcb.com/partdetail/DiodesIncorporated-AP63200WU7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
- U5: value ADS1115IDGS 0x48 -> ADS1115IDGSR 0x48; Purchase Link https://www.digikey.com/en/products/result?keywords=ADS1115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 -> https://jlcpcb.com/partdetail/TexasInstruments-ADS1115IDGSR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
- U6: value ADS1115IDGS 0x49 -> ADS1115IDGSR 0x49; Purchase Link https://www.digikey.com/en/products/result?keywords=ADS1115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 -> https://jlcpcb.com/partdetail/TexasInstruments-ADS1115IDGSR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
Connections:
- net +3V3_SW_LOGIC: now also D4.5 (REF2/+3V3), D5.5 (REF2/+3V3), D6.5 (REF2/+3V3), D7.5 (REF2/+3V3)
- net BATT_RAW_N: now also Q1.1 (S1); no longer C10.2, Q1.A1 (S1A), Q1.C1 (S1B)
- net CO_GATE: now also Q1.4 (G2); no longer Q1.B2 (G2)
- net DO_GATE: now also Q1.2 (G1); no longer Q1.B1 (G1)
- net EXP_GPA1: now also D4.3 (IO2); no longer D4.2 (IO2)
- net EXP_GPA3: now also D4.6 (IO4); no longer D4.5 (IO4)
- net EXP_GPA5: now also D5.3 (IO2); no longer D5.2 (IO2)
- net EXP_GPA7: now also D5.6 (IO4); no longer D5.5 (IO4)
- net EXP_GPB1: now also D6.3 (IO2); no longer D6.2 (IO2)
- net EXP_GPB3: now also D6.6 (IO4); no longer D6.5 (IO4)
- net EXP_GPB5: now also D7.3 (IO2); no longer D7.2 (IO2)
- net EXP_GPB7: now also D7.6 (IO4); no longer D7.5 (IO4)
- net GND: now also D4.2 (REF1/GND), D5.2 (REF1/GND), D6.2 (REF1/GND), D7.2 (REF1/GND), Q1.3 (S2); no longer D4.3 (GND), D5.3 (GND), D6.3 (GND), D7.3 (GND), J1.A12 (GND_A), Q1.A2 (S2A), Q1.C2 (S2B)
- new net Q1_DRAIN_COMMON: C10.2, J1.A12 (GND_A), Q1.5 (D1), Q1.6 (D1), Q1.7 (D2), Q1.8 (D2)
- no-connect marks 11 -> 7

Commit message: R14
Parts:
- removed Q1: PT8810 dual N-MOSFET, Package_SO:TSSOP-8_4.4x3mm_P0.65mm, symbol Daughterboard:PT8810_TSSOP8
- added C32, C33: 100nF 25V X7R, Capacitor_SMD:C_0603_1608Metric, symbol Daughterboard:TWO_PIN
- added Q1: CSD18502Q5B charge FET, Daughterboard:CSD18502Q5B_DNK0008A_VSON-CLIP_5x6mm, symbol Daughterboard:CSD18502Q5B
- added Q2: CSD18502Q5B discharge FET, Daughterboard:CSD18502Q5B_DNK0008A_VSON-CLIP_5x6mm, symbol Daughterboard:CSD18502Q5B
- added R49, R50: 10M, Resistor_SMD:R_0603_1608Metric, symbol Daughterboard:TWO_PIN
- added TP13: BATT_RAW_P test pad, TestPoint:TestPoint_Pad_D1.0mm, symbol Daughterboard:TESTPAD
- D1: value PESD5V0S1BA 5V VBUS TVS -> 5V VBUS TVS
- D4, D5, D6, D7: value SRV05-4.TCT / C13612 4ch ESD -> 4ch 3.3V GPIO TVS array TBD; footprint Package_TO_SOT_SMD:SOT-23-6 -> Daughterboard:SOT-23-6_NoPad6; Purchase Link https://jlcpcb.com/partdetail/Semtech-SRV05_4TCT/C13612 -> https://www.digikey.com/en/products/result?keywords=4+chann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
- F1: value BSMD1206-200-16V 2A hold polyfuse -> 2A hold polyfuse
- F2: value BSMD1206-200-16V cell1 PTC -> PTC/fuse cell1
- F3: value BSMD1206-200-16V cell2 PTC -> PTC/fuse cell2
- F4: value BSMD1206-200-16V system fuse -> 2A battery path fuse; Purchase Link https://www.digikey.com/en/products/result?keywords=2A+syst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 -> https://www.digikey.com/en/products/result?keywords=2A+batt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
- J4: value BM05B-GHS-TBT UART JST-GH top-entry 1.25mm -> UART JST-GH 1.25mm; footprint Connector_JST:JST_GH_BM05B-GHS-TBT_1x05-1MP_P1.25mm_Vertical -> Connector_JST:JST_GH_SM05B-GHS-TB_1x05-1MP_P1.25mm_Horizontal; Purchase Link https://jlcpcb.com/partdetail/JST-BM05BGHSTBTLF_SN_N/C189891 -> https://www.digikey.com/en/products/result?keywords=SM05B-G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
- J5: value I2C 2.54mm through-hole male header -> I2C male header 2.54mm; Purchase Link (none) -> https://www.digikey.com/en/products/result?keywords=2.54mm+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
- J6: value Deep sleep 2.54mm through-hole header -> Deep sleep pushbutton header; Purchase Link (none) -> https://www.digikey.com/en/products/result?keywords=2.54mm+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
- L3: value ANR5040T1R0M 1uH -> 1uH >=4A sat
- R3: Purchase Link https://jlcpcb.com/partdetail/C2692785 -> https://www.digikey.com/en/products/result?keywords=0603+re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
- R4: value 43R 1W CBSET -> TBD 1%; footprint Resistor_SMD:R_2512_6332Metric -> Resistor_SMD:R_0603_1608Metric; Purchase Link https://jlcpcb.com/partdetail/C38957 -> https://www.digikey.com/en/products/result?keywords=0603+re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
- TH1: value NCP18XH103F03RB 10k NTC -> 10k NTC
- TP3: value PACK_P test pad -> BAT_SYS test pad
- U1: value BQ25887RGER 2S charger -> BQ25887RGE 2S charger; Purchase Link https://jlcpcb.com/partdetail/TexasInstruments-BQ25887RGER/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 -> https://www.digikey.com/en/products/result?keywords=BQ25887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
- U3: value AP63200WU-7 5V Buck -> AP63200WU 5V Buck; Purchase Link https://jlcpcb.com/partdetail/DiodesIncorporated-AP63200WU7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 -> https://www.digikey.com/en/products/result?keywords=AP63200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
- U4: value AP63200WU-7 3V3 Buck -> AP63200WU 3V3 Buck; Purchase Link https://jlcpcb.com/partdetail/DiodesIncorporated-AP63200WU7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 -> https://www.digikey.com/en/products/result?keywords=AP63200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
- U5: value ADS1115IDGSR 0x48 -> ADS1115IDGS 0x48; Purchase Link https://jlcpcb.com/partdetail/TexasInstruments-ADS1115IDGSR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 -> https://www.digikey.com/en/products/result?keywords=ADS1115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
- U6: value ADS1115IDGSR 0x49 -> ADS1115IDGS 0x49; Purchase Link https://jlcpcb.com/partdetail/TexasInstruments-ADS1115IDGSR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 -> https://www.digikey.com/en/products/result?keywords=ADS1115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
Connections:
- net +3V3_SW_LOGIC: no longer D4.5 (REF2/+3V3), D5.5 (REF2/+3V3), D6.5 (REF2/+3V3), D7.5 (REF2/+3V3)
- net BATT_RAW_N: now also C10.2, R48.1; no longer R47.1
- net BAT_SYS: now also C5.1, TP3.1 (PAD), U1.13 (BAT1), U1.14 (BAT2), U1.15 (SNS1), U1.16 (SNS2), C32.1, Q1.5 (D), Q1.6 (D), Q1.7 (D), Q1.8 (D); no longer F4.2
- net CO_GATE: now also Q1.4 (G), R50.1
- net DO_GATE: now also Q2.4 (G), R49.1
- net EXP_GPA1: now also D4.2 (IO2); no longer D4.3 (IO2)
- net EXP_GPA3: now also D4.5 (IO4); no longer D4.6 (IO4)
- net EXP_GPA5: now also D5.2 (IO2); no longer D5.3 (IO2)
- net EXP_GPA7: now also D5.5 (IO4); no longer D5.6 (IO4)
- net EXP_GPB1: now also D6.2 (IO2); no longer D6.3 (IO2)
- net EXP_GPB3: now also D6.5 (IO4); no longer D6.6 (IO4)
- net EXP_GPB5: now also D7.2 (IO2); no longer D7.3 (IO2)
- net EXP_GPB7: now also D7.5 (IO4); no longer D7.6 (IO4)
- net GND: now also D4.3 (GND), D5.3 (GND), D6.3 (GND), D7.3 (GND), J1.A12 (GND_A), R47.1; no longer D4.2 (REF1/GND), D5.2 (REF1/GND), D6.2 (REF1/GND), D7.2 (REF1/GND), R48.1
- net CHG_IN renamed BATT_RAW_P
- net BATT_RAW_P: now also C9.1, F3.2, F4.2, J7.3, R14.1, TP13.1 (PAD)
- removed net PACK_P: C5.1, C9.1, F3.2, F4.1, J7.3, R14.1, TP3.1 (PAD), U1.13 (BAT1), U1.14 (BAT2), U1.15 (SNS1), U1.16 (SNS2)
- removed net Q1_DRAIN_COMMON: C10.2, J1.A12 (GND_A)
- new net FET_BATT_P: C33.1, F4.1, Q2.5 (D), Q2.6 (D), Q2.7 (D), Q2.8 (D)
- new net FET_SRC_COMMON: C32.2, C33.2, Q1.1 (S), Q1.2 (S), Q1.3 (S), Q2.1 (S), Q2.2 (S), Q2.3 (S), R49.2, R50.2
- no-connect marks 7 -> 11
