File: Hosyond_apr24b/Daughterboard/Daughterboard_before_nc_smd_pads_removed.kicad_sch (KiCad schematic)
At the start: 153 parts, among them J1 USB-C 5V Sink, J2 Switched power outputs, J30 J3P Hosyond +5V_SW solder pad, J31 J3A Hosyond UART_TX solder pad, J32 J3B Hosyond UART_RX solder pad, J33 J3C Hosyond I2C_SDA solder pad, J34 J3D Hosyond I2C_SCL solder pad, J35 J3E Hosyond GPIO2 solder pad, J36 J3F Hosyond GPIO3 solder pad, J37 J3G Hosyond GPIO14 solder pad, J38 J3H Hosyond GPIO21 solder pad, J39 J3I Hosyond GND solder pad, J4 UART JST-GH 1.25mm, J5 I2C male header 2.54mm, J6 Deep sleep pushbutton header, J7 2S balance input JST-XH, J8 Analog input header, J91 MCP23017 GPA0 solder pad, J910 MCP23017 GPB1 solder pad, J911 MCP23017 GPB2 solder pad, J912 MCP23017 GPB3 solder pad, J913 MCP23017 GPB4 solder pad, J914 MCP23017 GPB5 solder pad, J915 MCP23017 GPB6 solder pad, J916 MCP23017 GPB7 solder pad, J92 MCP23017 GPA1 solder pad, J925 MCP23017 INTA solder pad, J926 MCP23017 INTB solder pad, J927 MCP23017 RESET solder pad, J928 MCP23017 +3V3_SW solder pad, J929 MCP23017 GND solder pad, J93 MCP23017 GPA2 solder pad, J94 MCP23017 GPA3 solder pad, J95 MCP23017 GPA4 solder pad, J96 MCP23017 GPA5 solder pad, J97 MCP23017 GPA6 solder pad, J98 MCP23017 GPA7 solder pad, J99 MCP23017 GPB0 solder pad, Q1 CSD83325L, SW1 Pololu #2808 5V switch, SW2 Pololu #2808 3V3 switch, U1 BQ25887RGE 2S charger, U2 S-8252AAH-M6T1U, U3 AP63200WU 5V Buck, U4 AP63200WU 3V3 Buck, U5 ADS1115IDGS 0x48, U6 ADS1115IDGS 0x49, U7 MCP23017-E/SO

Commit message: k
Parts:
- removed R45: 0R, Resistor_SMD:R_0603_1608Metric, symbol Daughterboard:TWO_PIN
- C17: value 100nF 10V X7R DNP -> 100nF 10V X7R
- C8: now fitted
- D4, D5, D6, D7: value SP0504BAHTG 4ch GPIO TVS -> 4ch 3.3V GPIO TVS array TBD; footprint Daughterboard:SOT-23-6_NoPad6 -> Package_TO_SOT_SMD:SOT-23-6; Purchase Link https://www.digikey.com/en/products/result?keywords=SP0504B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 -> https://www.digikey.com/en/products/result?keywords=4+chann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
- R3: value 806R 1% ILIM -> 806R 1% TBD; Purchase Link https://www.digikey.com/en/products/result?keywords=806+ohm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 -> https://www.digikey.com/en/products/result?keywords=0603+re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
- R4: value 220R 1% CBSET -> TBD 1%; Purchase Link https://www.digikey.com/en/products/result?keywords=220+ohm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 -> https://www.digikey.com/en/products/result?keywords=0603+re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
- U7: footprint Daughterboard:SOIC-28W_7.5x17.9mm_P1.27mm_NoPads11_14 -> Package_SO:SOIC-28W_7.5x17.9mm_P1.27mm
Connections:
- net +3V3_SW_LOGIC is gone; now on net +3V3_SW: C17.1, C18.1, C19.1, C20.1, C27.1, C28.1, J928.1 (PAD), R19.2, R20.2, R42.1, R43.1, R44.1, U5.8 (VDD), U6.1 (ADDR), U6.8 (VDD), U7.9 (VDD)
- net CELL_MID: no longer R4.2
- net GND: now also R4.2
