File: Hosyond_apr24b/Daughterboard/Daughterboard_before_usb_j1_net_fix.kicad_pcb (KiCad board)
At the start: 4 copper layers, 155 x 80.6 mm, 150 parts, among them J1 USB-C 5V Sink, J30 J3P Hosyond +5V_SW solder pad, J31 J3A Hosyond UART_TX solder pad, J32 J3B Hosyond UART_RX solder pad, J33 J3C Hosyond I2C_SDA solder pad, J34 J3D Hosyond I2C_SCL solder pad, J35 J3E Hosyond GPIO2 solder pad, J36 J3F Hosyond GPIO3 solder pad, J37 J3G Hosyond GPIO14 solder pad, J38 J3H Hosyond GPIO21 solder pad, J39 J3I Hosyond GND solder pad, J4 UART JST-GH 1.25mm, J5 I2C male header 2.54mm, J6 Deep sleep pushbutton header, J7 2S balance input JST-XH, J8 Analog input header, J91 MCP23017 GPA0 solder pad, J910 MCP23017 GPB1 solder pad, J911 MCP23017 GPB2 solder pad, J912 MCP23017 GPB3 solder pad, J913 MCP23017 GPB4 solder pad, J914 MCP23017 GPB5 solder pad, J915 MCP23017 GPB6 solder pad, J916 MCP23017 GPB7 solder pad, J92 MCP23017 GPA1 solder pad, J925 MCP23017 INTA solder pad, J926 MCP23017 INTB solder pad, J927 MCP23017 RESET solder pad, J928 MCP23017 +3V3_SW solder pad, J929 MCP23017 GND solder pad, J93 MCP23017 GPA2 solder pad, J94 MCP23017 GPA3 solder pad, J95 MCP23017 GPA4 solder pad, J96 MCP23017 GPA5 solder pad, J97 MCP23017 GPA6 solder pad, J98 MCP23017 GPA7 solder pad, J99 MCP23017 GPB0 solder pad, Q1 CSD83325L, SW1 Pololu #2808 5V switch, SW2 Pololu #2808 3V3 switch, U1 BQ25887RGE 2S charger, U2 S-8252AAH-M6T1U, U3 AP63200WU 5V Buck, U4 AP63200WU 3V3 Buck, U5 ADS1115IDGS 0x48, U6 ADS1115IDGS 0x49, U7 MCP23017-E/SO

Commit message: k
Parts:
- removed J30: J3P Hosyond +5V_SW solder pad, TestPoint_Pad_1.5x1.5mm
- removed R45: 0R, R_0603_1608Metric
- C8: value 100nF 10V X7R DNP -> 100nF 10V X7R
- D4, D5, D6, D7: value SP0504BAHTG 4ch GPIO TVS -> 4ch 3.3V GPIO TVS array TBD; footprint SOT-23-6_NoPad6 -> SOT-23-6
- R3: value 806R 1% ILIM -> 806R 1% TBD
- R4: value 220R 1% CBSET -> TBD 1%
- U7: footprint SOIC-28W_7.5x17.9mm_P1.27mm_NoPads11_14 -> SOIC-28W_7.5x17.9mm_P1.27mm
- moved TP8 58.0 mm to (35.0, 66.0)
- moved R1 57.0 mm to (26.0, 13.0)
- moved R2 56.0 mm to (31.0, 13.0)
- moved R20 46.2 mm to (155.0, 54.0), turned to 0 degrees
- moved J910 41.6 mm to (122.0, 54.6)
- moved J911 40.5 mm to (124.5, 54.6)
- moved U5 40.1 mm to (124.5, 49.0), turned to 0 degrees
- moved U6 39.7 mm to (132.0, 49.0), turned to 0 degrees
- moved D4 35.8 mm to (129.5, 54.6), turned to 0 degrees
- moved J99 35.7 mm to (120.0, 50.0)
- moved TP2 35.6 mm to (20.0, 75.0)
- moved R18 35.4 mm to (55.0, 52.0)
- moved TP1 35.0 mm to (15.0, 75.0)
- moved TP6 34.9 mm to (15.0, 85.0)
- moved TP4 34.5 mm to (15.0, 80.0)
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Connections:
- C17 pad 1: +3V3_SW_LOGIC -> +3V3_SW
- C18 pad 1: +3V3_SW_LOGIC -> +3V3_SW
- C19 pad 1: +3V3_SW_LOGIC -> +3V3_SW
- C20 pad 1: +3V3_SW_LOGIC -> +3V3_SW
- C27 pad 1: +3V3_SW_LOGIC -> +3V3_SW
- C28 pad 1: +3V3_SW_LOGIC -> +3V3_SW
- J1 pad A12: GND -> (no net)
- J1 pad A5: CC1 -> (no net)
- J1 pad A9: USB_VBUS -> (no net)
- J1 pad B12: GND -> (no net)
- J1 pad B5: CC2 -> (no net)
- J1 pad B9: USB_VBUS -> (no net)
- J1 pad SH: GND -> (no net)
- J928 pad 1: +3V3_SW_LOGIC -> +3V3_SW
- R19 pad 2: +3V3_SW_LOGIC -> +3V3_SW
- R20 pad 2: +3V3_SW_LOGIC -> +3V3_SW
- R4 pad 2: CELL_MID -> GND
- R42 pad 1: +3V3_SW_LOGIC -> +3V3_SW
- R43 pad 1: +3V3_SW_LOGIC -> +3V3_SW
- R44 pad 1: +3V3_SW_LOGIC -> +3V3_SW
- U5 pad 8: +3V3_SW_LOGIC -> +3V3_SW
- U6 pad 1: +3V3_SW_LOGIC -> +3V3_SW
- U6 pad 8: +3V3_SW_LOGIC -> +3V3_SW
- U7 pad 9: +3V3_SW_LOGIC -> +3V3_SW
Routing:
- net +3V3_SW_LOGIC: track 173.2 -> 0.00 mm, vias 3 -> 0
- net +3V3_SW: track 108.4 -> 226.6 mm
- net CELL_MID: track 62.0 -> 148.3 mm, vias 4 -> 1
- net I2C_SDA: track 178.9 -> 252.3 mm
- net MCP_GPA0: track 5.63 -> 63.6 mm, vias 0 -> 2
- net CHG_IN: track 35.6 -> 79.0 mm, vias 0 -> 3
- net MCP_INTB: track 21.5 -> 63.6 mm, vias 2 -> 4
- net MCP_GPA5: track 5.21 -> 46.2 mm
- net BAT_SYS: track 129.9 -> 170.6 mm, vias 4 -> 5
- net GPIO3: track 31.9 -> 71.8 mm
- net MCP_GPB2: track 4.84 -> 42.8 mm, vias 0 -> 4
- net EXP_GPB4: track 69.2 -> 31.3 mm, vias 3 -> 2
- net MCP_INTA: track 25.0 -> 62.2 mm, vias 2 -> 3
- net AIN7: track 9.22 -> 44.8 mm
- net TS: track 14.1 -> 48.6 mm, vias 3 -> 4
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- added copper zone on B.Cu, net GND
- removed copper zone on In1.Cu, net GND
Other:
- copper layers 4 -> 2
